File: Chorus.sch (KiCad schematic (older format))
At the start: 104 parts, among them IC2 NJM4558, IC3 NE571, IC4 M5224P, IC5 MN3209, IC6 MN3102, IC7 M5224P, IC8 NJM2903, Q1 ?, Q2 ?, Q4 ?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

Commit message: Moved independent boards to sub-projects
Changed lines of the file:
@@
 $Descr User 7205 7481
 encoding utf-8
-Sheet 2 3
+Sheet 2 5
 Title ""
 Date ""
@@
 Comment4 ""
 $EndDescr
-$Sheet
-S 1100 2550 550  800
-U 59F87971
-F0 "Chorus_Extensions" 31
-F1 "Chorus_Extensions.sch" 31
-F2 "+A" I L 1100 2800 31
-F3 "-A" I L 1100 3000 31
-F4 "GND" I L 1100 2900 31
-F5 "DryRet" O R 1650 2700 31
-F6 "Dry" I L 1100 2600 31
-F7 "TriRet" O R 1650 3300 31
-F8 "Squ" I L 1100 3300 31
-F9 "SquRet" O L 1100 3200 31
-F10 "R" O R 1650 3100 31
-F11 "L" O R 1650 3200 31
-F12 "Tri" I L 1100 3100 31
-F13 "AuxJack" I L 1100 2700 31
-F14 "Wet" I R 1650 2600 31
-$EndSheet
 $Comp
 L CP1_Small C39
@@
 Text Notes 5650 950  0    39   ~ 8
 Post-Chorus Filtering
+$Sheet
+S 1100 2550 550  800
+U 59FAB4E6
+F0 "Chorus_Extensions" 31
+F1 "Chorus_Extensions.sch" 28
+F2 "-A" I L 1100 3000 35
+F3 "+A" I L 1100 2800 31
+F4 "GND" I L 1100 2900 31
+F5 "DryRet" O R 1650 2700 31
+F6 "Dry" I L 1100 2600 31
+F7 "TriRet" O R 1650 3300 31
+F8 "Squ" I L 1100 3300 31
+F9 "SquRet" O L 1100 3200 31
+F10 "R" O R 1650 3100 31
+F11 "L" O R 1650 3200 31
+F12 "Tri" I L 1100 3100 31
+F13 "AuxJack" I L 1100 2700 31
+F14 "Wet" I R 1650 2600 31
+$EndSheet
 $EndSCHEMATC
