File: Chorus.sch (KiCad schematic (older format))
At the start: 104 parts, among them IC2 NJM4558, IC3 NE571, IC4 M5224P, IC5 MN3209, IC6 MN3102, IC7 M5224P, IC8 NJM2903, Q1 ?, Q2 ?, Q4 ?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

Commit message: Chorus mod effectively complete sans some clean up
Connections:
- net Chorus_Mods/DryRet renamed ChorusMod/DryRet
- net Chorus_Mods/L renamed ChorusMod/L
- net Chorus_Mods/R renamed ChorusMod/R
- net Chorus_Mods/Squ renamed ChorusMod/Squ
- net Chorus_Mods/SquRet renamed ChorusMod/SquRet
- net Chorus_Mods/Tri renamed ChorusMod/Tri
- net Chorus_Mods/TriRet renamed ChorusMod/TriRet
- net Chorus_Mods/Wet renamed ChorusMod/Wet
Changed lines of the file:
@@
 $Descr User 7205 7481
 encoding utf-8
-Sheet 2 5
+Sheet 2 3
 Title ""
 Date ""
@@
 S 1100 2550 550  800
 U 59FAB4E6
-F0 "Chorus_Mods" 31
-F1 "Chorus_Mods.sch" 28
+F0 "ChorusMod" 31
+F1 "./ChorusMod/ChorusMod.sch" 24
 F2 "-A" I L 1100 3000 35
 F3 "+A" I L 1100 2800 31
