File: Chorus.sch (KiCad schematic (older format))
At the start: 104 parts, among them IC2 NJM4558, IC3 NE571, IC4 M5224P, IC5 MN3209, IC6 MN3102, IC7 M5224P, IC8 NJM2903, Q1 ?, Q2 ?, Q4 ?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

Commit message: save-point before some experimental pcb markings
Parts:
- IC2, IC8: symbol DualOpAmp -> Dual-Op-Amp
- IC4, IC7: symbol QuadOpAmp -> Quad-Op-Amp
- IC5: symbol BBD_Short -> BBD-Short
- IC6: symbol MN3102 -> BBD-Short-Clk
Connections:
- net labels removed: AuxJack
- wire segments 323 -> 322
Changed lines of the file:
@@
 EESchema Schematic File Version 2
+LIBS:Poly-800-rescue
 LIBS:power
 LIBS:device
@@
 LIBS:switches
 LIBS:MiscellaneousDevices
-LIBS:DualOpAmp
-LIBS:MN3102
-LIBS:NE571
-LIBS:QuadOpAmp
+LIBS:MyKi_Connectors
+LIBS:MyKi_Switches
+LIBS:MyKi_DIP_IC
+LIBS:MyKi_Board_Features
 LIBS:Poly-800-cache
 EELAYER 25 0
@@
 -A
 $Comp
-L BBD_Short IC5
+L BBD-Short IC5
 U 1 1 59F8B7EB
 P 5400 3050
@@
 $EndComp
 $Comp
-L MN3102 IC6
+L BBD-Short-Clk IC6
 U 1 1 59F8B8A9
 P 5400 4650
@@
 $EndComp
 $Comp
-L QuadOpAmp IC4
+L Quad-Op-Amp IC4
 U 1 1 59F95AC0
 P 1600 1550
@@
 Text HLabel 1050 2900 0    31   Input ~ 0
 GND
-Text HLabel 1050 2700 0    31   Input ~ 0
-AuxJack
 $Comp
 L R R30
@@
 	1    0    0    -1
 $EndComp
-Text HLabel 1050 2600 0    31   Input ~ 0
+Text HLabel 850  2700 0    31   Input ~ 0
 AudioIn
-Text Notes 750  2450 0    31   ~ 6
+Text Notes 600  2650 0    31   ~ 6
 aprox 1V PTP\nKorg's Input\nFET switching \nhas no effect\non signal and\nwas omitted.
 $Comp
@@
 Korg's output FET \nswitching has no\neffect on signal\nand was ommmited.
 $Comp
-L QuadOpAmp IC7
+L Quad-Op-Amp IC7
 U 1 1 5A10BE82
 P 1400 4200
@@
 $EndComp
 $Comp
-L DualOpAmp IC8
+L Dual-Op-Amp IC8
 U 1 1 5A181291
 P 2950 4400
@@
 +D
 $Comp
-L DualOpAmp IC2
+L Dual-Op-Amp IC2
 U 1 1 5A1B03E7
 P 2200 3150
@@
 	1050 2900 1100 2900
 Wire Wire Line
-	1050 2700 1100 2700
-Wire Wire Line
 	1150 850  1150 1450
 Wire Wire Line
@@
 Connection ~ 1900 5950
 Wire Wire Line
-	1050 2600 1100 2600
+	850  2700 1100 2700
 Text HLabel 1900 6350 2    31   Output ~ 0
 -D
@@
 F4 "GND" I L 1100 2900 31
 F5 "DryRet" O R 1650 2700 31
-F6 "Dry" I L 1100 2600 31
+F6 "Dry" I L 1100 2700 31
 F7 "TriRet" O R 1650 3300 31
 F8 "Squ" I L 1100 3300 31
@@
 F11 "L" O R 1650 3200 31
 F12 "Tri" I L 1100 3100 31
-F13 "AuxJack" I L 1100 2700 31
-F14 "Wet" I R 1650 2600 31
+F13 "Wet" I R 1650 2600 31
 $EndSheet
 $EndSCHEMATC

Commit message: Chorus mod effectively done sans some cleanup
Connections:
- net Chorus_Mods/DryRet renamed ChorusMod/DryRet
- net Chorus_Mods/L renamed ChorusMod/L
- net Chorus_Mods/R renamed ChorusMod/R
- net Chorus_Mods/Squ renamed ChorusMod/Squ
- net Chorus_Mods/SquRet renamed ChorusMod/SquRet
- net Chorus_Mods/Tri renamed ChorusMod/Tri
- net Chorus_Mods/TriRet renamed ChorusMod/TriRet
- net Chorus_Mods/Wet renamed ChorusMod/Wet
Other:
- note added: "<- Compressor Output"
- note added: "<- Signal to Expander"
- note added: "<- Wet Signal From Expander"
- note added: "Aprox 1V PTP."
- note added: "Dry Signal Input to compressor ->"
- note added: "Envelope Detection"
- note added: "Korg's Input\nFET switching\n(used to mute\nwhen synth\nis inactive) \nhas no effect\non signal and\nwas omitted."
- note added: "This may work with F1 for noise suppression.\nIf so, it should probably be omitted somehow."
- note added: "Wet Signal->"
- note removed: "aprox 1V PTP\nKorg's Input\nFET switching \nhas no effect\non signal and\nwas omitted."
- note removed: "compressor Input"
- note removed: "compressor Output"
- moved on the sheet: C27, C28, D2, D3, D4, D5, IC4, R35, R36, R37, R38, R39
