File: Chorus_Extensions.sch (KiCad schematic (older format))
At the start: 64 parts, among them SW1 ChorusFilterPan, SW2 AuxToChorus, SW3 Chorus-FilterPan-B, SW4 KorgToChorus, SW5 ChorusFbInv, SW6 Chorus-Fb_Invert-B, SW7 LFO2 Sel, U1 TL084, U2 NJM4556

Commit message: Moved independent boards to sub-projects
Parts:
- removed C1, C3, C4: 47n, symbol C_Small
- removed C11, C17, C47, C48, C49, C51, C6: 0.1µ, symbol C_Small
- removed C14, C15: 10µ, symbol CP1_Small
- removed C20: 1µ, symbol C_Small
- removed C21, C26, C5, C50, C7: 1µ, symbol CP1_Small
- removed D1, D8: 2v2, symbol D_Zener_Small_ALT
- removed D7, D9: 1N4148, symbol D_ALT
- removed R1, R5, R6: 22K, symbol R
- removed R10, R11: 5.1K, symbol R
- removed R12, R13: 47K, symbol R
- removed R14, R78: 100K, symbol R
- removed R15, R19, R8, R9: 470, symbol R
- removed R17, R77: 1.5M, symbol R
- removed R18, R7: 1K, symbol R
- removed R2, R27, R28: 33K, symbol R
- removed R23, R25: 18K, symbol R
- removed R59: 10K, symbol R
- removed R61: 4.7K, symbol R
- removed R74: 12K, symbol R
- removed R75: 1M, symbol R
- removed R76: 220K, symbol R
- removed RV1: DUAL_B250K, symbol POT_Dual
- removed RV2, RV3: B100K, symbol POT
- removed RV4: DUAL_B100K, symbol POT_Dual
- removed RV5: B1M, symbol POT
- removed RV6: B10K, symbol POT
- removed SW1: ChorusFilterPan, symbol SW_DPDT_x2
- removed SW2: AuxToChorus, symbol SW_DPDT_x2
- removed SW3: Chorus-FilterPan-B, symbol SW_DPDT_x2
- removed SW4: KorgToChorus, symbol SW_DPDT_x2
- removed SW5: ChorusFbInv, symbol SW_DPDT_x2
- removed SW6: Chorus-Fb_Invert-B, symbol SW_DPDT_x2
- removed SW7: LFO2 Sel, symbol SW_SPDT
- removed U1: TL084, MODULE, symbol QuadOpAmp
- removed U2: NJM4556, MODULE, symbol DualOpAmp
Connections:
- net labels removed: DryOut, DryR, Fb, WetL, WetR
- wire segments 186 -> 22
Other:
- note removed: "(wire)"
- note removed: "<- to HPF w/Ω\n(norm. Right)"
- note removed: "<- to LPF (norm.\nLeft) and Fb"
- note removed: "<-Left\nChannel Wet \n(normally LP)"
- note removed: "<-Right \nChannel Wet \n(normally HP)"
- note removed: "Aux \nInput \nTrim"
- note removed: "Aux. In Buffer"
- note removed: "Aux. Input\nVoltage\nProtection"
- note removed: "Bias Correction"
- note removed: "Chorus Input Active Mixer"
- note removed: "Chorus Input Switches"
- note removed: "Chorus LFO \nOutput Buffer"
- note removed: "Chorus \nStereo \nSeparation"
- note removed: "Chorus-Control PCB"
- note removed: "Chorus-Extension PCB"
- note removed: "Chorus\nDepth"
- note removed: "Chorus\nFeedback"
- note removed: "Chorus\nRate"
- note removed: "Chorus\nWetPass"
- note removed: "Feedback's \ngain is limited\nby LP filtering"
- note removed: "From top edge\nof PCB at R47"
- note removed: "GND"
- note removed: "GND from \ntop edge\nof PCB at \nC42 neg"
- note removed: "Glued to right of KLM-598 and bolted to synth \ncase with preexisting unused scew holes."
- note removed: "HP Wet"
- note removed: "Inv"
- note removed: "LP Wet"
- note removed: "Not Filtered,\n possibly\n Inverted"
- note removed: "PCB mounted pots on\nChorus-Control PCB"
- note removed: "Point to Point Wiring \nmounted left of \nChorus In switches"
- note removed: "Point to Point Wiring below Upper RIght PCB"
- note removed: "Point to Point \nWiring mounted \nbelow Chorus \nDepth and Rate"
- note removed: "Point to Point wiring right\nof Chorus-Control PCB\n"
- note removed: "Replacement of C26 which \n was 0.47µ"
- note removed: "Replaces\nKorg's \nC20,\nno need \nfor it on\nLP"
- note removed: "Square LFO from removed \nR61 on pin14 of IC7 side"
- note removed: "Square LFO from removed \nR61 on pin9 of IC7 side"
- note removed: "The L & R channel \nfeedback resistors \non main chorus \nboard op amp IC2, \nR24 & R22 repectively, \nshould both be replaced \nwith 33K resistors."
- note removed: "This is Korg's C15, just moved out."
- note removed: "To left side of removed \nR28 on Korg"
- note removed: "To left side of removed\nR27 on Korg"
- note removed: "Triangle LFO from \nremoved R59 on \npin8 of IC7 side"
- note removed: "Triangle LFO from\nremoved R59 on \npin6 of IC7 side"
- note removed: "Wet"
- note removed: "Wet from \nremoved\nC20"
- note removed: "Wet-Inverted"
- note removed: "dry from removed \nC15 on Korg, F1 side"
- note removed: "from R48 \nat top edge\nof PCB"
- note removed: "mounted to synth's upper right edge\nvia pots attachement to the synth"
- note removed: "norm"
- note removed: "to removed C15 \ntoward IC3 pin6"
- note removed: "|"
