File: Poly-800_mod.sch (KiCad schematic (older format))
At the start: 0 parts

Commit message: Moved independent boards to sub-projects
Changed lines of the file:
@@
 $Descr User 10157 6103
 encoding utf-8
-Sheet 1 3
+Sheet 1 5
 Title "Poly-800 Extensions"
 Date "2017-10-29"
@@
 $EndDescr
 $Sheet
-S 5100 950  1050 750
-U 59F878A4
+S 5050 2450 950  400
+U 59FAABE9
 F0 "Chorus" 31
 F1 "Chorus.sch" 31
