File: Chorus_Mods.sch (KiCad schematic (older format))
At the start: 0 parts

Commit message: save-point before some experimental pcb markings
Changed lines of the file:
@@
 EESchema Schematic File Version 2
+LIBS:Poly-800-rescue
 LIBS:power
 LIBS:device
@@
 LIBS:switches
 LIBS:MiscellaneousDevices
-LIBS:DualOpAmp
-LIBS:MN3102
-LIBS:NE571
-LIBS:QuadOpAmp
+LIBS:MyKi_Connectors
+LIBS:MyKi_Switches
+LIBS:MyKi_DIP_IC
+LIBS:MyKi_Board_Features
 LIBS:Poly-800-cache
 EELAYER 25 0
@@
 Tri
 Text HLabel 800  1850 0    39   Input ~ 0
-AuxJack
-Text HLabel 800  1950 0    39   Input ~ 0
 Wet
 $Sheet
-S 900  650  750  1400
+S 900  650  750  1300
 U 59FAE5D3
 F0 "Chorus_Ext" 39
@@
 F11 "L" O L 900 1650 31
 F12 "Tri" I L 900 1750 31
-F13 "AuxJack" I L 900 1850 31
-F14 "Dry→" O R 1650 750 31
-F15 "WetL←" I R 1650 850 31
-F16 "DryR←" I R 1650 950 31
-F17 "WetR←" I R 1650 1050 31
-F18 "+A→" O R 1650 1150 31
-F19 "GND→" O R 1650 1250 31
-F20 "-A→" O R 1650 1350 31
-F21 "FB←" I R 1650 1450 31
-F22 "Wet→" O R 1650 1550 31
-F23 "Wet" I L 900 1950 31
+F13 "Dry→" O R 1650 750 31
+F14 "WetL←" I R 1650 850 31
+F15 "DryR←" I R 1650 950 31
+F16 "WetR←" I R 1650 1050 31
+F17 "+A→" O R 1650 1150 31
+F18 "GND→" O R 1650 1250 31
+F19 "-A→" O R 1650 1350 31
+F20 "FB←" I R 1650 1450 31
+F21 "Wet→" O R 1650 1550 31
+F22 "Wet" I L 900 1850 31
 $EndSheet
 $Sheet
@@
 	800  1850 900  1850
 Wire Wire Line
-	800  1950 900  1950
-Wire Wire Line
 	1650 750  2000 750

Commit message: routine  save-point
Changed lines of the file:
@@
 LIBS:MyKi_DIP_IC
 LIBS:MyKi_Board_Features
+LIBS:MyKI_Potentiometers
 LIBS:Poly-800-cache
 EELAYER 25 0
 EELAYER END
-$Descr User 5118 4724
+$Descr User 5315 4724
 encoding utf-8
 Sheet 3 5
@@
 Comment4 ""
 $EndDescr
-Text HLabel 800  750  0    39   Input ~ 0
+Text HLabel 800  1050 0    39   Input ~ 0
 +A
 Text HLabel 800  950  0    39   Input ~ 0
 -A
-Text HLabel 800  850  0    39   Input ~ 0
+Text HLabel 800  1150 0    39   Input ~ 0
 GND
-Text HLabel 800  1050 0    39   Output ~ 0
+Text HLabel 800  850  0    39   Output ~ 0
 DryRet
-Text HLabel 800  1150 0    39   Input ~ 0
+Text HLabel 800  750  0    39   Input ~ 0
 Dry
-Text HLabel 800  1250 0    39   Output ~ 0
+Text HLabel 800  1850 0    39   Output ~ 0
 TriRet
-Text HLabel 800  1350 0    39   Input ~ 0
+Text HLabel 800  1550 0    39   Input ~ 0
 Squ
+Text HLabel 800  1650 0    39   Output ~ 0
+SquRet
+Text HLabel 800  1350 0    39   Output ~ 0
+R
 Text HLabel 800  1450 0    39   Output ~ 0
-SquRet
-Text HLabel 800  1550 0    39   Output ~ 0
-R
-Text HLabel 800  1650 0    39   Output ~ 0
 L
 Text HLabel 800  1750 0    39   Input ~ 0
 Tri
-Text HLabel 800  1850 0    39   Input ~ 0
+Text HLabel 800  1250 0    39   Input ~ 0
 Wet
-$Sheet
-S 900  650  750  1300
-U 59FAE5D3
-F0 "Chorus_Ext" 39
-F1 "./Chorus_Ext/Chorus_Ext.sch" 29
-F2 "+A" I L 900 750 31
-F3 "-A" I L 900 950 31
-F4 "GND" I L 900 850 31
-F5 "DryRet" O L 900 1050 31
-F6 "Dry" I L 900 1150 31
-F7 "TriRet" O L 900 1250 31
-F8 "Squ" I L 900 1350 31
-F9 "SquRet" O L 900 1450 31
-F10 "R" O L 900 1550 31
-F11 "L" O L 900 1650 31
-F12 "Tri" I L 900 1750 31
-F13 "Dry→" O R 1650 750 31
-F14 "WetL←" I R 1650 850 31
-F15 "DryR←" I R 1650 950 31
-F16 "WetR←" I R 1650 1050 31
-F17 "+A→" O R 1650 1150 31
-F18 "GND→" O R 1650 1250 31
-F19 "-A→" O R 1650 1350 31
-F20 "FB←" I R 1650 1450 31
-F21 "Wet→" O R 1650 1550 31
-F22 "Wet" I L 900 1850 31
-$EndSheet
-$Sheet
-S 2000 650  750  1150
-U 59FAE7A0
-F0 "Chorus_Ctrl" 39
-F1 "./Chorus_Ctrl/Chorus_Ctrl.sch" 29
-F2 "Wet" I L 2000 1550 31
-F3 "Dry" I L 2000 750 31
-F4 "WetL" O L 2000 850 31
-F5 "DryR" O L 2000 950 31
-F6 "WetR" O L 2000 1050 31
-F7 "+A" I L 2000 1150 31
-F8 "GND" I L 2000 1250 31
-F9 "-A" I L 2000 1350 31
-F10 "FB" O L 2000 1450 31
-$EndSheet
 Text Notes 4100 2200 0    31   ~ 0
 Stereo\n  Pot
@@
 Wire Wire Line
 	1650 1550 2000 1550
+$Sheet
+S 900  700  750  1200
+U 5A11371F
+F0 "Chorus_Ext" 31
+F1 "./Chorus_Ext/Chorus_Ext.sch" 31
+F2 "+A_A4" I L 900 1050 31
+F3 "-A_A3" I L 900 950 31
+F4 "GND_A5" I L 900 1150 31
+F5 "DryRet_A2" O L 900 850 31
+F6 "Dry_A1" I L 900 750 31
+F7 "Dry_B1" O R 1650 750 31
+F8 "WetL_B2" I R 1650 850 31
+F9 "DryR_B3" I R 1650 950 31
+F10 "WetR_B4" I R 1650 1050 31
+F11 "+A_B6" O R 1650 1250 31
+F12 "GND_B7" O R 1650 1350 31
+F13 "-A_B8" O R 1650 1450 31
+F14 "FB_B9" I R 1650 1550 31
+F15 "Wet_B5" O R 1650 1150 31
+F16 "Wet_A6" I L 900 1250 31
+F17 "TriRet_A4" O L 900 1850 31
+F18 "Squ_A1" I L 900 1550 31
+F19 "SquRet_A2" O L 900 1650 31
+F20 "R_A7" O L 900 1350 31
+F21 "L_A8" O L 900 1450 31
+F22 "Tri_A3" I L 900 1750 31
+$EndSheet
+$Sheet
+S 2000 700  750  1000
+U 5A113D17
+F0 "Chorus_Ctrl" 31
+F1 "./Chorus_Ctrl/Chorus_Ctrl.sch" 31
+F2 "Wet" I L 2000 1150 31
+F3 "Dry" I L 2000 750 31
+F4 "WetL" O L 2000 850 31
+F5 "DryR" O L 2000 950 31
+F6 "WetR" O L 2000 1050 31
+F7 "+A" I L 2000 1250 31
+F8 "GND" I L 2000 1350 31
+F9 "-A" I L 2000 1450 31
+F10 "FB" O L 2000 1550 31
+$EndSheet
 $EndSCHEMATC
