File: ChorusMod.kicad_pcb (KiCad board)
At the start: 2 copper layers, 119 parts, among them J1 AuxAudioIn, J1.11 WT, J1.12 BK, J1.13 OR, J1.14 YL, J1.15 OR+BK, J1.16 YL+BK, J1.17 GN, J2.1 BN, J2.2 RD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

Commit message: save point after modding my Korg. Next: replace wire colors with meaningful labels others can follow
Parts:
- moved W1.1 50.9 mm to (129.5, 78.7)
- moved W1.2 48.5 mm to (127.0, 78.7)
- moved SW6 30.0 mm to (134.0, 91.4)
- moved SW3 20.3 mm to (113.0, 91.4), turned to 270 degrees
- moved R14 13.0 mm to (116.8, 101.6), turned to 90 degrees
- moved J1.14 10.2 mm to (124.5, 73.7)
- moved SW5 7.10 mm to (102.9, 91.4), turned to 270 degrees
- moved J1.17 5.68 mm to (124.5, 78.7)
- moved SW4 3.05 mm to (124.5, 91.4), turned to 270 degrees
Connections:
- W1.7 pad 2: Net-(J1.7-Pad2) -> /Squ
Routing:
- net Net-(J1.12-Pad2): track 0.00 -> 66.5 mm
- net Net-(R77-Pad1): track 0.00 -> 51.4 mm
- net Net-(J1.14-Pad2): track 0.00 -> 50.0 mm
- net Net-(R76-Pad2): track 0.00 -> 44.6 mm
- net Net-(R14-Pad1): track 0.00 -> 27.0 mm
- net Net-(J1.13-Pad2): track 0.00 -> 25.7 mm
- net Net-(J1.11-Pad2): track 0.00 -> 23.4 mm
- net Net-(J1.16-Pad2): track 0.00 -> 20.9 mm
- net Net-(J1.15-Pad2): track 0.00 -> 19.4 mm
- net Net-(J1.17-Pad2): track 0.00 -> 19.2 mm
- net Net-(C26-Pad1): track 20.6 -> 7.62 mm
- net Net-(J1.17-Pad1): track 5.08 -> 10.8 mm
- net Net-(J1.7-Pad2): track 0.00 -> 0.63 mm
