File: Chorus_Ext/_saved_Chorus_Ext.sch (KiCad schematic (older format))
At the start: 46 parts, among them SW2 AuxToChorus, SW4 KorgToChorus, SW7 LFO2 Sel, U1 TL084

Commit message: further work on pcb
Parts:
- C1, C3, C4, C47, C6: footprint MyKicadPath:200Mil_TH_C -> MyKi_TH_Capacitors:200Mil_TH_C
- C14, C15, C26, C5, C50: footprint MyKicadPath:200Mil_TH_CP -> MyKi_TH_Capacitors:200Mil_TH_CP
- D1, D7, D8, D9: footprint MyKicadPath:400Mil_TH_Diode -> MyKi_TH_Diodes:400Mil_TH_Diode
- R1, R11, R14, R15, R2, R23, R25, R27, R28, R5, R59, R6, R61, R76, R77, R78, R9: footprint MyKicadPath:400Mil_TH_Resistor -> MyKi_TH_Resistors:400Mil_TH_Resistor
- R10, R17, R19, R74, R75, R8: footprint MyKicadPath:300Mil_TH_Resistor -> MyKi_TH_Resistors:300Mil_TH_Resistor
- R18, R7: footprint MyKicadPath:400Mil_TH_Resistor -> MyKi_TH_Resistors:300Mil_TH_Resistor
- RV2, RV3, RV5: footprint MyKicadPath:Potentiometer_Alps-RK16-single -> MyKi_TH_Panel_Controls:Potentiometer_Alps-RK16-single
- U1: footprint MyKicadPath:300Mil_TH_DIP14 -> MyKi_TH_IC:300Mil_TH_DIP14
