File: Chorus_Ext/Chorus_Ext.kicad_pcb (KiCad board)
At the start: 2 copper layers, 53.3 x 73.7 mm, 56 parts, among them SW2 AuxToChorus, SW4 KorgToChorus, SW7 LFO2 Sel, U1 TL084

Commit message: further work on pcb
Parts:
- removed the D9 at (57.1, 106.6)
- added D9: 1N4148, MyKicadPath:400Mil_TH_Diode, F.Cu at (15.2, 48.3)
- added D9: 1N4148, MyKi_TH_Diodes:400Mil_TH_Diode, F.Cu at (50.8, 73.7)
- C1, C3, C4, C47, C6: footprint Capacitors_THT:C_Disc_D4.3mm_W1.9mm_P5.00mm -> MyKi_TH_Capacitors:200Mil_TH_C
- C14, C15, C26, C5, C50: footprint Capacitors_THT:CP_Radial_D5.0mm_P2.50mm -> MyKi_TH_Capacitors:200Mil_TH_CP
- D1, D7, D8: footprint Diodes_THT:D_DO-41_SOD81_P7.62mm_Horizontal -> MyKi_TH_Diodes:400Mil_TH_Diode
- R1, R11, R14, R15, R2, R23, R25, R27, R28, R5, R59, R6, R61, R76, R77, R78, R9: footprint Resistors_THT:R_Axial_DIN0207_L6.3mm_D2.5mm_P7.62mm_Horizontal -> MyKi_TH_Resistors:400Mil_TH_Resistor
- R10, R17, R18, R19, R7, R74, R75, R8: footprint Resistors_THT:R_Axial_DIN0207_L6.3mm_D2.5mm_P7.62mm_Horizontal -> MyKi_TH_Resistors:300Mil_TH_Resistor
- RV2, RV3, RV5: footprint MyKicadPath:Potentiometer_Alps-RK16-single -> MyKi_TH_Panel_Controls:Potentiometer_Alps-RK16-single
- U1: footprint Housings_DIP:DIP-14_W7.62mm_Socket -> MyKi_TH_IC:300Mil_TH_DIP14
- moved SW4 79.0 mm to (96.5, 38.1)
- moved SW2 72.5 mm to (96.5, 45.7)
- moved R76 68.0 mm to (111.8, 66.0), turned to 270 degrees
- moved R28 68.0 mm to (40.6, 40.6)
- moved C26 66.1 mm to (53.3, 40.6), turned to 90 degrees
- moved RV3 65.8 mm to (99.1, 55.9)
- moved R23 65.5 mm to (40.6, 43.2)
- moved C3 64.4 mm to (68.6, 43.2), turned to 270 degrees
- moved C4 64.0 mm to (66.0, 43.2), turned to 270 degrees
- moved C1 63.7 mm to (63.5, 43.2), turned to 270 degrees
- moved R27 63.1 mm to (40.6, 45.7)
- moved R25 60.6 mm to (40.6, 48.3)
- moved C5 58.2 mm to (40.6, 50.8), turned to 270 degrees
- moved R14 57.5 mm to (43.2, 50.8)
- moved R2 57.0 mm to (68.6, 50.8), turned to 270 degrees
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Other:
- board outline removed

Commit message: save-point before some experimental pcb markings
Parts:
- removed the D9 at (15.2, 48.3)
- added J1: AuxAudioIn, w_conn_av:rca_red, F.Cu at (39.9, 53.3)
- added JP1: Dry, MyKi_TH_Board_Features:TH_Via, F.Cu at (53.3, 38.1)
- added JP10: Aux→Sw, MyKi_TH_Board_Features:TH_Via, F.Cu at (76.2, 61.0)
- added JP11: Aux←Sw, MyKi_TH_Board_Features:TH_Via, F.Cu at (83.8, 40.6)
- added JP12: Korg←Sw, MyKi_TH_Board_Features:TH_Via, F.Cu at (81.3, 40.6)
- added JP13: PotGND, MyKi_TH_Board_Features:TH_Via, F.Cu at (88.9, 68.6)
- added JP14: LFO2, MyKi_TH_Board_Features:TH_Via, F.Cu at (71.1, 91.4)
- added JP15: AuxIn, MyKi_TH_Board_Features:TH_Via, F.Cu at (53.3, 71.1)
- added JP16: AuxGND, MyKi_TH_Board_Features:TH_Via, F.Cu at (53.3, 68.6)
- added JP17: Squ, MyKi_TH_Board_Features:TH_Via, F.Cu at (103.6, 74.5)
- added JP18: SquRet, MyKi_TH_Board_Features:TH_Via, F.Cu at (103.1, 81.5)
- added JP19: Tri, MyKi_TH_Board_Features:TH_Via, F.Cu at (96.5, 101.6)
- added JP2: DryRet, MyKi_TH_Board_Features:TH_Via, F.Cu at (88.9, 58.4)
- added JP20: TriRet, MyKi_TH_Board_Features:TH_Via, F.Cu at (103.4, 69.5)
- added JP3: -A, MyKi_TH_Board_Features:TH_Via, F.Cu at (53.3, 88.9)
- added JP4: +A, MyKi_TH_Board_Features:TH_Via, F.Cu at (53.3, 53.3)
- added JP5: GND, MyKi_TH_Board_Features:TH_Via, F.Cu at (53.3, 86.4)
- added JP6: Wet, MyKi_TH_Board_Features:TH_Via, F.Cu at (66.0, 50.8)
- added JP7: R, MyKi_TH_Board_Features:TH_Via, F.Cu at (53.3, 45.7)
- added JP8: L, MyKi_TH_Board_Features:TH_Via, F.Cu at (53.3, 43.2)
- added JP9: Korg→Sw, MyKi_TH_Board_Features:TH_Via, F.Cu at (68.6, 35.6)
- added P1: Wet→, MyKi_TH_Board_Features:TH_Via, F.Cu at (71.1, 50.8)
- added P2: Dry→, MyKi_TH_Board_Features:TH_Via, F.Cu at (71.1, 40.6)
- added P3: →FB, MyKi_TH_Board_Features:TH_Via, F.Cu at (76.2, 43.2)
- added P4: WetL←, MyKi_TH_Board_Features:TH_Via, F.Cu at (71.1, 43.2)
- added P5: DryR←, MyKi_TH_Board_Features:TH_Via, F.Cu at (71.1, 45.7)
- added P6: WetR←, MyKi_TH_Board_Features:TH_Via, F.Cu at (71.1, 48.3)
- added P7: +A→, MyKi_TH_Board_Features:TH_Via, F.Cu at (71.1, 53.3)
- added P8: GND, MyKi_TH_Board_Features:TH_Via, F.Cu at (76.2, 53.3)
- added P9: -A, MyKi_TH_Board_Features:TH_Via, F.Cu at (76.2, 45.7)
- A1, A18, X1, X18: renamed from REF**; footprint MyKicadPath:BackPlated_TH -> MyKi_TH_Board_Features:BackPlated_TH
- C14, C15, C26, C5, C50: footprint MyKi_TH_Capacitors:200Mil_TH_CP -> MyKi_TH_Capacitors:100Mil_TH_CP
- Drill1, Drill2: renamed from REF**; footprint MyKicadPath:3mm_DrillHole -> MyKi_TH_Board_Features:3mm_DrillHole
- Hole1, Hole2, Hole3, Hole4: renamed from REF**; footprint MyKicadPath:2mm_DrillHole -> MyKi_TH_Board_Features:2mm_DrillHole
- R14, R5, R59, R61, R76, R77: footprint MyKi_TH_Resistors:400Mil_TH_Resistor -> MyKi_TH_Resistors:300Mil_TH_Resistor
- RV2, RV3, RV5: footprint MyKi_TH_Panel_Controls:Potentiometer_Alps-RK16-single -> MyKi_TH_Panel_Controls:Pot_TH_Mini_pcbEdge
- SW2, SW4, SW7: footprint Buttons_Switches_THT:SW_Micro_SPST -> w_switch:switch_mfp116dg-ra
- U1: footprint MyKi_TH_IC:300Mil_TH_DIP14 -> MyKi_TH_IC:300Mil_DIP14
- moved R76 38.3 mm to (100.3, 102.6), turned to 90 degrees
- moved C14 31.8 mm to (39.9, 61.0), turned to 270 degrees
- moved R14 28.4 mm to (71.1, 55.9), turned to 270 degrees
- moved RV2 24.6 mm to (43.7, 68.6)
- moved R61 24.4 mm to (113.0, 80.0), turned to 180 degrees
- moved R78 18.3 mm to (68.6, 81.3), turned to 270 degrees
- moved R77 17.3 mm to (100.3, 83.6)
- moved C15 16.1 mm to (86.4, 58.4)
- moved R10 16.1 mm to (73.7, 68.6), turned to 90 degrees
- moved SW7 15.5 mm to (113.0, 89.9), turned to 90 degrees
- moved C5 15.5 mm to (55.9, 53.3)
- moved A1 15.2 mm to (94.0, 94.0)
- moved D7 15.2 mm to (66.0, 58.4)
- moved D9 15.2 mm to (66.0, 73.7)
- moved Drill1 15.2 mm to (90.4, 41.7)
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Connections:
- net /+A renamed Net-(C5-Pad1)
- net /-A renamed Net-(C47-Pad1)
- net /Dry→ renamed Net-(C26-Pad1)
- net /L renamed Net-(JP8-Pad2)
- net /R renamed Net-(JP7-Pad2)
- net /Squ renamed Net-(JP17-Pad2)
- net /Tri renamed Net-(JP19-Pad2)
- net Net-(C15-Pad2) renamed /ToChorus
- C1 pad 1: /FB← -> Net-(C1-Pad1)
- C14 pad 1: /AuxJack -> Net-(C14-Pad1)
- C15 pad 1: /DryRet -> Net-(C15-Pad1)
- C26 pad 2: /Dry -> Net-(C26-Pad2)
- R10 pad 2: Net-(R10-Pad2) -> Net-(JP10-Pad1)
- R11 pad 1: Net-(R11-Pad1) -> Net-(JP15-Pad2)
- R23 pad 2: /WetL← -> Net-(P4-Pad1)
- R25 pad 2: /WetR← -> Net-(P6-Pad1)
- R27 pad 2: /DryR← -> Net-(P5-Pad1)
- R59 pad 2: /TriRet -> Net-(JP20-Pad2)
- R61 pad 2: /SquRet -> Net-(JP18-Pad2)
- R75 pad 1: Net-(R75-Pad1) -> Net-(JP14-Pad1)
- RV2 pad 1: Net-(C14-Pad2) -> Net-(J1-Pad2)
- RV2 pad 2: Net-(R11-Pad1) -> Net-(JP15-Pad1)
- RV2 pad 3: /GND -> Net-(C14-Pad2)
- RV3 pad 1: /GND -> Net-(JP13-Pad2)
- SW2 pad 1: Net-(R10-Pad2) -> Net-(SW2-Pad1)
- SW2 pad 2: Net-(C3-Pad1) -> Net-(JP11-Pad2)
- SW4 pad 1: /Dry -> Net-(SW4-Pad1)
- SW4 pad 2: Net-(C4-Pad1) -> Net-(JP12-Pad2)
- SW7 pad 2: Net-(R75-Pad1) -> Net-(JP14-Pad2)
- U1 pad 1: Net-(R10-Pad2) -> Net-(JP10-Pad1)
Routing:
- net /GND: track 0.00 -> 121.3 mm
- net Net-(C47-Pad1): track 0.00 -> 103.5 mm
- net Net-(JP19-Pad2): track 0.00 -> 56.2 mm
- net Net-(C5-Pad1): track 0.00 -> 46.5 mm
- net Net-(JP10-Pad2): track 0.00 -> 40.3 mm
- net Net-(JP9-Pad2): track 0.00 -> 39.2 mm
- net Net-(JP14-Pad2): track 0.00 -> 33.2 mm
- net Net-(JP11-Pad2): track 0.00 -> 31.3 mm
- net Net-(J1-Pad2): track 0.00 -> 29.7 mm
- net Net-(JP12-Pad2): track 0.00 -> 25.6 mm
- net Net-(JP13-Pad2): track 0.00 -> 22.2 mm
- net Net-(C26-Pad2): track 0.00 -> 15.6 mm
- net Net-(R1-Pad1): track 0.00 -> 15.6 mm
- net Net-(D7-Pad1): track 0.00 -> 15.2 mm
- net Net-(D9-Pad2): track 0.00 -> 15.2 mm
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Other:
- board text added: "Control-PCB Jumper Wires"

Commit message: just a save-point
Parts:
- removed JP1: Dry, MyKi_TH_Board_Features:TH_Via
- removed JP10: Aux→Sw, MyKi_TH_Board_Features:TH_Via
- removed JP11: Aux←Sw, MyKi_TH_Board_Features:TH_Via
- removed JP12: Korg←Sw, MyKi_TH_Board_Features:TH_Via
- removed JP13: PotGND, MyKi_TH_Board_Features:TH_Via
- removed JP14: LFO2, MyKi_TH_Board_Features:TH_Via
- removed JP15: AuxIn, MyKi_TH_Board_Features:TH_Via
- removed JP16: AuxGND, MyKi_TH_Board_Features:TH_Via
- removed JP17: Squ, MyKi_TH_Board_Features:TH_Via
- removed JP18: SquRet, MyKi_TH_Board_Features:TH_Via
- removed JP19: Tri, MyKi_TH_Board_Features:TH_Via
- removed JP2: DryRet, MyKi_TH_Board_Features:TH_Via
- removed JP20: TriRet, MyKi_TH_Board_Features:TH_Via
- removed JP3, P9: -A, MyKi_TH_Board_Features:TH_Via
- removed JP4: +A, MyKi_TH_Board_Features:TH_Via
- removed JP5, P8: GND, MyKi_TH_Board_Features:TH_Via
- removed JP6: Wet, MyKi_TH_Board_Features:TH_Via
- removed JP7: R, MyKi_TH_Board_Features:TH_Via
- removed JP8: L, MyKi_TH_Board_Features:TH_Via
- removed JP9: Korg→Sw, MyKi_TH_Board_Features:TH_Via
- removed P1: Wet→, MyKi_TH_Board_Features:TH_Via
- removed P2: Dry→, MyKi_TH_Board_Features:TH_Via
- removed P3: →FB, MyKi_TH_Board_Features:TH_Via
- removed P4: WetL←, MyKi_TH_Board_Features:TH_Via
- removed P5: DryR←, MyKi_TH_Board_Features:TH_Via
- removed P6: WetR←, MyKi_TH_Board_Features:TH_Via
- removed P7: +A→, MyKi_TH_Board_Features:TH_Via
- added P_+A_A4: red, MyKi_TH_Connectors:TH_Wire_unlabeled, F.Cu at (53.3, 53.3)
- added P_+A_B6: red, MyKi_TH_Connectors:Conn_Female_Dupont-1_Val, F.Cu at (71.1, 53.3)
- added P_-A_A3: brown, MyKi_TH_Connectors:TH_Wire_unlabeled, F.Cu at (53.3, 88.9)
- added P_-A_B8: brown, MyKi_TH_Connectors:Conn_Female_Dupont-1_Val, F.Cu at (73.7, 45.7)
- added P_Aux_P2: orange, MyKi_TH_Connectors:Conn_Female_Dupont-1_Val, F.Cu at (76.2, 61.0)
- added P_Aux_P3: orange+b, MyKi_TH_Connectors:Conn_Female_Dupont-1_Val, F.Cu at (83.8, 40.6)
- added P_Aux_P7: orange, MyKi_TH_Connectors:Conn_Female_Dupont-1_Val, F.Cu at (53.3, 71.1)
- added P_DryR_B3: orange+b, MyKi_TH_Connectors:Conn_Female_Dupont-1_Val, F.Cu at (71.1, 45.7)
- added P_DryRet_A2: green, MyKi_TH_Connectors:TH_Wire_unlabeled, F.Cu at (88.9, 58.4)
- added P_Dry_A1: yellow, MyKi_TH_Connectors:TH_Wire_unlabeled, F.Cu at (53.3, 38.1)
- added P_Dry_B1: orange, MyKi_TH_Connectors:Conn_Female_Dupont-1_Val, F.Cu at (71.1, 40.6)
- added P_FB_B9: green, MyKi_TH_Connectors:Conn_Female_Dupont-1_Val, F.Cu at (73.7, 43.2)
- added P_GND_A5: black, MyKi_TH_Connectors:TH_Wire_unlabeled, F.Cu at (53.3, 86.4)
- added P_GND_B7: black, MyKi_TH_Connectors:Conn_Female_Dupont-1_Val, F.Cu at (73.7, 53.3)
- added P_GND_P5: black, MyKi_TH_Connectors:Conn_Female_Dupont-1_Val, F.Cu at (88.9, 68.6)
- added P_GND_P8: black, MyKi_TH_Connectors:Conn_Female_Dupont-1_Val, F.Cu at (53.3, 68.6)
- added P_KS_P1: yellow, MyKi_TH_Connectors:Conn_Female_Dupont-1_Val, F.Cu at (68.6, 35.6)
- added P_KS_P4: yellow+b, MyKi_TH_Connectors:Conn_Female_Dupont-1_Val, F.Cu at (81.3, 40.6)
- added P_LFO_P6: white, MyKi_TH_Connectors:Conn_Female_Dupont-1_Val, F.Cu at (71.1, 91.4)
- added P_L_A8: yellow, MyKi_TH_Connectors:TH_Wire_unlabeled, F.Cu at (53.3, 43.2)
- added P_R_A7: orange, MyKi_TH_Connectors:TH_Wire_unlabeled, F.Cu at (53.3, 48.3)
- added P_WetL_B3: yellow, MyKi_TH_Connectors:Conn_Female_Dupont-1_Val, F.Cu at (71.1, 43.2)
- added P_WetR_B4: purple, MyKi_TH_Connectors:Conn_Female_Dupont-1_Val, F.Cu at (71.1, 48.3)
- added P_Wet_A6: blue, MyKi_TH_Connectors:TH_Wire_unlabeled, F.Cu at (66.0, 50.8)
- added P_Wet_B5: blue, MyKi_TH_Connectors:Conn_Female_Dupont-1_Val, F.Cu at (71.1, 50.8)
- added W_SquRet_A2: white+b, MyKi_TH_Connectors:Wire_Ref-Val, F.Cu at (103.9, 81.3)
- added W_Squ_A1: white, MyKi_TH_Connectors:Wire_Ref-Val, F.Cu at (102.6, 72.4)
- added W_TriRet_A4: grey+b, MyKi_TH_Connectors:Wire_Ref-Val, F.Cu at (100.3, 73.2)
- added W_Tri_A3: grey, MyKi_TH_Connectors:Wire_Ref-Val, F.Cu at (97.5, 102.6)
Connections:
- net /GND renamed Net-(C47-Pad2)
Routing:
- net Net-(P_Wet_A6-Pad1): track 0.00 -> 5.08 mm
- net Net-(JP6-Pad2): track 4.57 -> 0.00 mm
- net Net-(C1-Pad1): track 2.29 -> 5.08 mm
- net Net-(C47-Pad2): track 121.3 -> 123.9 mm
- net Net-(C5-Pad1): track 46.5 -> 49.1 mm
- net Net-(C47-Pad1): track 103.5 -> 105.9 mm
- net Net-(R77-Pad2): track 14.6 -> 13.1 mm
- net Net-(R59-Pad2): track 3.12 -> 1.91 mm
- net Net-(R61-Pad2): track 2.54 -> 1.80 mm
Other:
- board text added: "Control-PCB"
- board text removed: "Control-PCB Jumper Wires"

Commit message: routine  save-point
Parts:
- removed P_WetL_B3: yellow, MyKi_TH_Connectors:Conn_Female_Dupont-1_Val
- added P_WetL_B2: yellow, MyKi_TH_Connectors:Conn_Female_Dupont-1_Val, F.Cu at (71.1, 43.2)
- P_+A_A4, P_-A_A3, P_DryRet_A2, P_Dry_A1, P_GND_A5, P_L_A8, P_R_A7, P_Wet_A6: footprint MyKi_TH_Connectors:TH_Wire_unlabeled -> MyKi_TH_Connectors:TH_Wire_Val
- SW3: renamed from SW4; value KorgToChorus -> AuxToChorus
- SW4: renamed from SW2; value AuxToChorus -> KorgToChorus
- moved W_Tri_A3 42.4 mm to (103.9, 60.7)
- moved R76 22.7 mm to (113.0, 83.8), turned to 180 degrees
- moved SW3 16.8 mm to (110.5, 49.5)
- moved SW4 16.5 mm to (110.5, 32.8)
- moved R77 15.0 mm to (100.3, 98.6)
- moved P_Dry_A1 7.62 mm to (61.0, 38.1)
- moved SW5 4.20 mm to (114.8, 93.7)
- renumbered P_Dry_B1 to P_DryCP_B1, RV3 to RV4, RV2 to RV6, SW7 to SW5
Connections:
- SW3 pad 2: Net-(P_KS_P4-Pad2) -> Net-(P_Aux_P3-Pad2)
- SW3 pad 3: Net-(P_KS_P1-Pad2) -> Net-(P_Aux_P2-Pad2)
- SW4 pad 2: Net-(P_Aux_P3-Pad2) -> Net-(P_KS_P4-Pad2)
- SW4 pad 3: Net-(P_Aux_P2-Pad2) -> Net-(P_KS_P1-Pad2)
- SW5 pad 1: Net-(R76-Pad2) -> Net-(R77-Pad1)
- SW5 pad 3: Net-(R77-Pad1) -> Net-(R76-Pad2)
Routing:
- net Net-(R76-Pad1): track 56.2 -> 33.4 mm
- net Net-(R77-Pad2): track 13.1 -> 27.0 mm
- net Net-(C26-Pad2): track 15.6 -> 8.00 mm
- net Net-(P_LFO_P6-Pad2): track 33.2 -> 35.1 mm
- net Net-(R77-Pad1): track 3.86 -> 5.01 mm
- net Net-(R76-Pad2): track 4.60 -> 5.26 mm
- net (no net): track 0.00 -> 0.54 mm
