File: Chorus_Ext/Chorus_Ext.sch (KiCad schematic (older format))
At the start: 46 parts, among them SW2 AuxToChorus, SW4 KorgToChorus, SW7 LFO2 Sel, U1 TL084

Commit message: assign footprints, start pcb
Parts:
- C1, C3, C4, C47, C6: footprint (none) -> Capacitors_THT:C_Disc_D4.3mm_W1.9mm_P5.00mm
- C14, C15, C26, C5, C50: footprint (none) -> Capacitors_THT:CP_Radial_D5.0mm_P2.50mm
- D1, D7, D8, D9: footprint (none) -> Diodes_THT:D_DO-41_SOD81_P7.62mm_Horizontal
- R1, R10, R11, R14, R15, R17, R18, R19, R2, R23, R25, R27, R28, R5, R59, R6, R61, R7, R74, R75, R76, R77, R78, R8, R9: footprint (none) -> Resistors_THT:R_Axial_DIN0207_L6.3mm_D2.5mm_P7.62mm_Horizontal
- RV2, RV3, RV5: footprint (none) -> MyKicadPath:Potentiometer_Alps-RK16-single
- SW2, SW4, SW7: footprint (none) -> Buttons_Switches_THT:SW_Micro_SPST
- U1: footprint MODULE -> Housings_DIP:DIP-14_W7.62mm_Socket
Other:
- note added: "- - -"
- note added: "- - - -"
- note added: "Aux2Fx\n SW"
- note added: "Chorus\nControl\n PCB"
- note added: "Chorus\nExtension\n PCB"
- note added: "Depth\n Pot"
- note added: "FbInv\n SW"
- note added: "Feedback\n Pot"
- note added: "FiltPan\n SW"
- note added: "KLM-598-3\n PCB"
- note added: "Keyboard Keys"
- note added: "LFOShape\n SW"
- note added: "Rate\n Pot"
- note added: "Stereo\n Pot"
- note added: "Synth2Fx\n SW"
- note added: "WetPass\n Pot"

Commit message: further work on pcb
Parts:
- C1, C3, C4, C47, C6: footprint Capacitors_THT:C_Disc_D4.3mm_W1.9mm_P5.00mm -> MyKicadPath:200Mil_TH_C
- C14, C15, C26, C5, C50: footprint Capacitors_THT:CP_Radial_D5.0mm_P2.50mm -> MyKicadPath:200Mil_TH_CP
- D1, D7, D8, D9: footprint Diodes_THT:D_DO-41_SOD81_P7.62mm_Horizontal -> MyKicadPath:400Mil_TH_Diode
- R1, R11, R14, R15, R2, R23, R25, R27, R28, R5, R59, R6, R61, R76, R77, R78, R9: footprint Resistors_THT:R_Axial_DIN0207_L6.3mm_D2.5mm_P7.62mm_Horizontal -> MyKicadPath:400Mil_TH_Resistor
- R10, R17, R18, R19, R7, R74, R75, R8: footprint Resistors_THT:R_Axial_DIN0207_L6.3mm_D2.5mm_P7.62mm_Horizontal -> MyKicadPath:300Mil_TH_Resistor
- U1: footprint Housings_DIP:DIP-14_W7.62mm_Socket -> MyKicadPath:300Mil_TH_DIP14

Commit message: previously forgot to save before commit
Parts:
- C1, C3, C4, C47, C6: footprint MyKicadPath:200Mil_TH_C -> MyKi_TH_Capacitors:200Mil_TH_C
- C14, C15, C26, C5, C50: footprint MyKicadPath:200Mil_TH_CP -> MyKi_TH_Capacitors:200Mil_TH_CP
- D1, D7, D8, D9: footprint MyKicadPath:400Mil_TH_Diode -> MyKi_TH_Diodes:400Mil_TH_Diode
- R1, R11, R14, R15, R2, R23, R25, R27, R28, R5, R59, R6, R61, R76, R77, R78, R9: footprint MyKicadPath:400Mil_TH_Resistor -> MyKi_TH_Resistors:400Mil_TH_Resistor
- R10, R17, R18, R19, R7, R74, R75, R8: footprint MyKicadPath:300Mil_TH_Resistor -> MyKi_TH_Resistors:300Mil_TH_Resistor
- RV2, RV3, RV5: footprint MyKicadPath:Potentiometer_Alps-RK16-single -> MyKi_TH_Panel_Controls:Potentiometer_Alps-RK16-single
- U1: footprint MyKicadPath:300Mil_TH_DIP14 -> MyKi_TH_IC:300Mil_TH_DIP14

Commit message: save-point before some experimental pcb markings
Parts:
- added J1: AuxAudioIn, w_conn_av:rca_red, symbol TS_Jack
- added JP1: Dry, MyKi_TH_Board_Features:TH_Via, symbol Jumper_Wire
- added JP10: Aux→Sw, MyKi_TH_Board_Features:TH_Via, symbol Jumper_Wire
- added JP11: Aux←Sw, MyKi_TH_Board_Features:TH_Via, symbol Jumper_Wire
- added JP12: Korg←Sw, MyKi_TH_Board_Features:TH_Via, symbol Jumper_Wire
- added JP13: PotGND, MyKi_TH_Board_Features:TH_Via, symbol Jumper_Wire
- added JP14: LFO2, MyKi_TH_Board_Features:TH_Via, symbol Jumper_Wire
- added JP15: AuxIn, MyKi_TH_Board_Features:TH_Via, symbol Jumper_Wire
- added JP16: AuxGND, MyKi_TH_Board_Features:TH_Via, symbol Jumper_Wire
- added JP17: Squ, MyKi_TH_Board_Features:TH_Via, symbol Jumper_Wire
- added JP18: SquRet, MyKi_TH_Board_Features:TH_Via, symbol Jumper_Wire
- added JP19: Tri, MyKi_TH_Board_Features:TH_Via, symbol Jumper_Wire
- added JP2: DryRet, MyKi_TH_Board_Features:TH_Via, symbol Jumper_Wire
- added JP20: TriRet, MyKi_TH_Board_Features:TH_Via, symbol Jumper_Wire
- added JP3: -A, MyKi_TH_Board_Features:TH_Via, symbol Jumper_Wire
- added JP4: +A, MyKi_TH_Board_Features:TH_Via, symbol Jumper_Wire
- added JP5: GND, MyKi_TH_Board_Features:TH_Via, symbol Jumper_Wire
- added JP6: Wet, MyKi_TH_Board_Features:TH_Via, symbol Jumper_Wire
- added JP7: R, MyKi_TH_Board_Features:TH_Via, symbol Jumper_Wire
- added JP8: L, MyKi_TH_Board_Features:TH_Via, symbol Jumper_Wire
- added JP9: Korg→Sw, MyKi_TH_Board_Features:TH_Via, symbol Jumper_Wire
- added P1: Wet→, MyKi_TH_Board_Features:TH_Via, symbol Pad
- added P2: Dry→, MyKi_TH_Board_Features:TH_Via, symbol Pad
- added P3: FB←, MyKi_TH_Board_Features:TH_Via, symbol Pad
- added P4: WetL←, MyKi_TH_Board_Features:TH_Via, symbol Pad
- added P5: DryR←, MyKi_TH_Board_Features:TH_Via, symbol Pad
- added P6: WetR←, MyKi_TH_Board_Features:TH_Via, symbol Pad
- added P7: +A→, MyKi_TH_Board_Features:TH_Via, symbol Pad
- added P8: GND→, MyKi_TH_Board_Features:TH_Via, symbol Pad
- added P9: -A→, MyKi_TH_Board_Features:TH_Via, symbol Pad
- C14, C15, C26, C5, C50: footprint MyKi_TH_Capacitors:200Mil_TH_CP -> MyKi_TH_Capacitors:100Mil_TH_CP
- R14, R5, R59, R61, R76, R77: footprint MyKi_TH_Resistors:400Mil_TH_Resistor -> MyKi_TH_Resistors:300Mil_TH_Resistor
- RV2, RV3: footprint MyKi_TH_Panel_Controls:Potentiometer_Alps-RK16-single -> MyKi_TH_Panel_Controls:Pot_TH_Mini_pcbEdge
- RV5: footprint MyKi_TH_Panel_Controls:Potentiometer_Alps-RK16-single -> MyKi_TH_Panel_Controls:Pot_TH_Mini_pcbEdge; Parameter (none) -> Chorus Rate
- SW2, SW4, SW7: footprint Buttons_Switches_THT:SW_Micro_SPST -> w_switch:switch_mfp116dg-ra
- U1: footprint MyKi_TH_IC:300Mil_TH_DIP14 -> MyKi_TH_IC:300Mil_DIP14; symbol QuadOpAmp -> Quad-Op-Amp
Connections:
- net labels added: ToChorus
- net labels removed: AuxJack
- wire segments 128 -> 137
Other:
- note added: "Aux. Input Line Level Clipping"
- note added: "Bias\nCorrection"
- note added: "Chorus Input Mixer Inputs"
- note added: "Chorus LFO(2) \n/--Output Buffer--|"
- note added: "Jumper wires JP1 - JP8\nrun between Korg's \nKLM-598-3 pcb and this (Chorus-Ext) board. \nOne of these, JP4, is simply forwarded out to \nthe other chorus mod board: Chorus-Ctrl"
- note added: "Jumper wires JP17 - JP20 connect to point to point \nwired panel components directly to KLM-598-3\n"
- note added: "Jumper wires JP9 - JP16 connect directly between \npoint to point wired panel components arranged \naround the synth clockwise starting in upper right."
- note added: "Point to Point Wiring"
- note added: "Solder pads P1 - P9 connect to \njumper wires on the Chorus-Clrl board."
- note added: "Wet from \nremoved\nC20 (top)"
- note added: "to removed C15 \ntoward IC3 pin6"
- note added: "|--Aux. In Buffer--|"
- note added: "|-Chorus Input Mixer->"
- note removed: "Aux \nInput \nTrim"
- note removed: "Aux. In Buffer"
- note removed: "Aux. Input\nVoltage\nProtection"
- note removed: "Bias Correction"
- note removed: "Chorus Input Active Mixer"
- note removed: "Chorus LFO \nOutput Buffer"
- note removed: "From top edge\nof PCB at R47"
- note removed: "Point to Point Wiring \nmounted left of \nChorus In switches"
- note removed: "to removed \nC15 toward\nIC3 pin6"
- moved on the sheet: C14, C26, C47, C5, C50, R23, R25, R27, R28, R59, R61, R77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

Commit message: just a save-point
Parts:
- removed JP1: Dry, MyKi_TH_Board_Features:TH_Via, symbol Jumper_Wire
- removed JP10: Aux→Sw, MyKi_TH_Board_Features:TH_Via, symbol Jumper_Wire
- removed JP11: Aux←Sw, MyKi_TH_Board_Features:TH_Via, symbol Jumper_Wire
- removed JP12: Korg←Sw, MyKi_TH_Board_Features:TH_Via, symbol Jumper_Wire
- removed JP13: PotGND, MyKi_TH_Board_Features:TH_Via, symbol Jumper_Wire
- removed JP14: LFO2, MyKi_TH_Board_Features:TH_Via, symbol Jumper_Wire
- removed JP15: AuxIn, MyKi_TH_Board_Features:TH_Via, symbol Jumper_Wire
- removed JP16: AuxGND, MyKi_TH_Board_Features:TH_Via, symbol Jumper_Wire
- removed JP17: Squ, MyKi_TH_Board_Features:TH_Via, symbol Jumper_Wire
- removed JP18: SquRet, MyKi_TH_Board_Features:TH_Via, symbol Jumper_Wire
- removed JP19: Tri, MyKi_TH_Board_Features:TH_Via, symbol Jumper_Wire
- removed JP2: DryRet, MyKi_TH_Board_Features:TH_Via, symbol Jumper_Wire
- removed JP20: TriRet, MyKi_TH_Board_Features:TH_Via, symbol Jumper_Wire
- removed JP3: -A, MyKi_TH_Board_Features:TH_Via, symbol Jumper_Wire
- removed JP4: +A, MyKi_TH_Board_Features:TH_Via, symbol Jumper_Wire
- removed JP5: GND, MyKi_TH_Board_Features:TH_Via, symbol Jumper_Wire
- removed JP6: Wet, MyKi_TH_Board_Features:TH_Via, symbol Jumper_Wire
- removed JP7: R, MyKi_TH_Board_Features:TH_Via, symbol Jumper_Wire
- removed JP8: L, MyKi_TH_Board_Features:TH_Via, symbol Jumper_Wire
- removed JP9: Korg→Sw, MyKi_TH_Board_Features:TH_Via, symbol Jumper_Wire
- added P_+A_A4: red, MyKi_TH_Connectors:TH_Wire_unlabeled, symbol TH-Wire
- added P_-A_A3: brown, MyKi_TH_Connectors:TH_Wire_unlabeled, symbol TH-Wire
- added P_Aux_P2: orange, MyKi_TH_Connectors:Conn_Female_Dupont-1_Val, symbol F-M-Pins
- added P_Aux_P3: orange+b, MyKi_TH_Connectors:Conn_Female_Dupont-1_Val, symbol F-M-Pins
- added P_Aux_P7: orange, MyKi_TH_Connectors:Conn_Female_Dupont-1_Val, symbol TH-Wire
- added P_DryRet_A2: green, MyKi_TH_Connectors:TH_Wire_unlabeled, symbol TH-Wire
- added P_Dry_A1, P_L_A8: yellow, MyKi_TH_Connectors:TH_Wire_unlabeled, symbol TH-Wire
- added P_GND_A5: black, MyKi_TH_Connectors:TH_Wire_unlabeled, symbol TH-Wire
- added P_GND_P5: black, MyKi_TH_Connectors:Conn_Female_Dupont-1_Val, symbol F-M-Pins
- added P_GND_P8: black, MyKi_TH_Connectors:Conn_Female_Dupont-1_Val, symbol TH-Wire
- added P_KS_P1: yellow, MyKi_TH_Connectors:Conn_Female_Dupont-1_Val, symbol F-M-Pins
- added P_KS_P4: yellow+b, MyKi_TH_Connectors:Conn_Female_Dupont-1_Val, symbol F-M-Pins
- added P_LFO_P6: white, MyKi_TH_Connectors:Conn_Female_Dupont-1_Val, symbol F-M-Pins
- added P_R_A7: orange, MyKi_TH_Connectors:TH_Wire_unlabeled, symbol TH-Wire
- added P_Wet_A6: blue, MyKi_TH_Connectors:TH_Wire_unlabeled, symbol TH-Wire
- added W_SquRet_A2: white+b, MyKi_TH_Connectors:Wire_Ref-Val, symbol Wire
- added W_Squ_A1: white, MyKi_TH_Connectors:Wire_Ref-Val, symbol Wire
- added W_TriRet_A4: grey+b, MyKi_TH_Connectors:Wire_Ref-Val, symbol Wire
- added W_Tri_A3: grey, MyKi_TH_Connectors:Wire_Ref-Val, symbol Wire
- P_+A_B6: renamed from P7; value +A→ -> red; footprint MyKi_TH_Board_Features:TH_Via -> MyKi_TH_Connectors:Conn_Female_Dupont-1_Val; symbol Pad -> F-M-Pins
- P_-A_B8: renamed from P9; value -A→ -> brown; footprint MyKi_TH_Board_Features:TH_Via -> MyKi_TH_Connectors:Conn_Female_Dupont-1_Val; symbol Pad -> F-M-Pins
- P_DryR_B3: renamed from P5; value DryR← -> orange+b; footprint MyKi_TH_Board_Features:TH_Via -> MyKi_TH_Connectors:Conn_Female_Dupont-1_Val; symbol Pad -> F-M-Pins
- P_Dry_B1: renamed from P2; value Dry→ -> orange; footprint MyKi_TH_Board_Features:TH_Via -> MyKi_TH_Connectors:Conn_Female_Dupont-1_Val; symbol Pad -> F-M-Pins
- P_FB_B9: renamed from P3; value FB← -> green; footprint MyKi_TH_Board_Features:TH_Via -> MyKi_TH_Connectors:Conn_Female_Dupont-1_Val; symbol Pad -> F-M-Pins
- P_GND_B7: renamed from P8; value GND→ -> black; footprint MyKi_TH_Board_Features:TH_Via -> MyKi_TH_Connectors:Conn_Female_Dupont-1_Val; symbol Pad -> F-M-Pins
- P_WetL_B3: renamed from P4; value WetL← -> yellow; footprint MyKi_TH_Board_Features:TH_Via -> MyKi_TH_Connectors:Conn_Female_Dupont-1_Val; symbol Pad -> F-M-Pins
- P_WetR_B4: renamed from P6; value WetR← -> purple; footprint MyKi_TH_Board_Features:TH_Via -> MyKi_TH_Connectors:Conn_Female_Dupont-1_Val; symbol Pad -> F-M-Pins
- P_Wet_B5: renamed from P1; value Wet→ -> blue; footprint MyKi_TH_Board_Features:TH_Via -> MyKi_TH_Connectors:Conn_Female_Dupont-1_Val; symbol Pad -> F-M-Pins
Connections:
- net at C5.1, C6.2, P_+A_B6.1 (B)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: now also P_+A_A4.1
- net at C3.1: now also P_Aux_P3.1 (B)
- net at C15.1: now also P_DryRet_A2.1
- net at SW2.2 (B): now also P_Aux_P3.2 (F)
- net at SW2.3 (C): now also P_Aux_P2.2 (F)
- net at C47.1, C50.2, P_-A_B8.1 (B)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: now also P_-A_A3.1
- net at R11.1: now also P_Aux_P7.1
- net at J1.2 (S), RV2.1: now also P_GND_P8.2
- net at RV2.2: now also P_Aux_P7.2
- net at R10.2, U1.1 (←1): now also P_Aux_P2.1 (B)
- net at C4.1: now also P_KS_P4.1 (B)
- net at R75.1: now also P_LFO_P6.1 (B)
- net at R77.2, RV5.3: now also W_Squ_A1.2
- net at R61.2: now also W_SquRet_A2.2
- net at RV3.1: now also P_GND_P5.2 (F)
- net at R76.1, RV3.3: now also W_Tri_A3.2
- net at R59.2: now also W_TriRet_A4.2
- net at SW7.2 (B): now also P_LFO_P6.2 (F)
- net at SW4.2 (B): now also P_KS_P4.2 (F)
- net at SW4.3 (C): now also P_KS_P1.2 (F)
- net at R23.1, R28.1: now also P_L_A8.1
- net at R25.1, R27.1: now also P_R_A7.1
- net at C26.2: now also P_Dry_A1.1, P_KS_P1.1 (B)
- net at P_Wet_B5.1 (B): now also P_Wet_A6.1
- net +A→ renamed +A_B6
- net -A→ renamed -A_B8
- net DryR← renamed DryR_B3
- net Dry→ renamed Dry_B1
- net FB← renamed FB_B9
- net GND: no longer names the net of C47.2, C5.2, C50.1, C6.1, D1.2 (A), D8.1 (K), P_GND_B7.1 (B), R15.2, R9.1, U1.12 (4+)
- net GND: now also P_GND_A5.1, P_GND_P5.1 (B), P_GND_P8.1
- net GND→ renamed GND_B7
- net WetL← renamed WetL_B2
- net WetR← renamed WetR_B4
- net Wet→ renamed Wet_B5
- new net +A_A4: P_+A_A4.2
- new net -A_A3: P_-A_A3.2
- new net DryRet_A2: P_DryRet_A2.2
- new net Dry_A1: P_Dry_A1.2
- new net GND_A5: P_GND_A5.2
- new net L_A8: P_L_A8.2
- new net R_A7: P_R_A7.2
- new net SquRet_A2: W_SquRet_A2.1
- new net Squ_A1: W_Squ_A1.1
- new net TriRet_A4: W_TriRet_A4.1
- new net Tri_A3: W_Tri_A3.1
- new net Wet_A6: P_Wet_A6.2
Other:
- note added: "Ribbon B to\nCho-Ctrl PCB"
- note added: "Square LFO from \nremoved R61 on \npin9 of IC7 side"
- note added: "TH-Vias J_*_A* run between this \nChorus-Ext board and Korg's KLM-598-3."
- note added: "TH-Vias J_*_B* run this (Cho-Ext) board\nand the Cho-Ctrl board."
- note added: "TH-Vias J_*_P* connect directly between \npoint to point wired panel components arranged \naround the synth clockwise starting in upper right."
- note added: "The L & R channel \nfeedback resistors \non main chorus \nboard op amp IC2, \nR24 & R22 repectively, \nshould both be \nreplaced with 33K resistors."
- note added: "Wires W_*_A*connect point-to-point \nwired panel components directly to KLM-598-3\n"
- note added: "from removed C20 (top)"
- note removed: "Jumper wires JP1 - JP8\nrun between Korg's \nKLM-598-3 pcb and this (Chorus-Ext) board. \nOne of these, JP4, is simply forwarded out to \nthe other chorus mod board: Chorus-Ctrl"
- note removed: "Jumper wires JP17 - JP20 connect to point to point \nwired panel components directly to KLM-598-3\n"
- note removed: "Jumper wires JP9 - JP16 connect directly between \npoint to point wired panel components arranged \naround the synth clockwise starting in upper right."
- note removed: "Solder pads P1 - P9 connect to \njumper wires on the Chorus-Clrl board."
- note removed: "Square LFO from removed \nR61 on pin9 of IC7 side"
- note removed: "The L & R channel \nfeedback resistors \non main chorus \nboard op amp IC2, \nR24 & R22 repectively, \nshould both be replaced \nwith 33K resistors."
- note removed: "Wet from \nremoved\nC20 (top)"
- note removed: "to Chorus\nControl PCB"
- moved on the sheet: C14, C26, C47, J1, R23, R25, R27, R28, R59, R61, R76, R77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

Commit message: routine  save-point
Parts:
- P_+A_A4, P_-A_A3, P_DryRet_A2, P_Dry_A1, P_GND_A5, P_L_A8, P_R_A7, P_Wet_A6: footprint MyKi_TH_Connectors:TH_Wire_unlabeled -> MyKi_TH_Connectors:TH_Wire_Val
- SW2, SW4: symbol SW_DPDT_x2 -> SPDT
- SW7: symbol SW_SPDT -> SPDT
- renumbered P_Dry_B1 to P_DryCP_B1, P_WetL_B3 to P_WetL_B2
Connections:
- net at SW7.1 (off): now also R77.1; no longer R76.2
- net at SW7.3 (on): now also R76.2; no longer R77.1
Other:
- note added: "Header Pins P_*_B* run this (Cho-Ext) board\nand the Cho-Ctrl board."
- note added: "Header Pins P_*_P* connect directly between \npoint to point wired panel components arranged \naround the synth clockwise starting in upper right, \nwith *P1-*P6 being one ribbon and the remaining \ntwo as another."
- note added: "Pads P_*_A* run wires between this \nChorus-Ext board and Korg's KLM-598-3."
- note added: "Wires W_*_A* connect point-to-point \nwired panel components directly to KLM-598-3\n"
- note removed: "TH-Vias J_*_A* run between this \nChorus-Ext board and Korg's KLM-598-3."
- note removed: "TH-Vias J_*_B* run this (Cho-Ext) board\nand the Cho-Ctrl board."
- note removed: "TH-Vias J_*_P* connect directly between \npoint to point wired panel components arranged \naround the synth clockwise starting in upper right."
- note removed: "Wires W_*_A*connect point-to-point \nwired panel components directly to KLM-598-3\n"
