File: Chorus_Ctrl/Chorus_Ctrl.sch (KiCad schematic (older format))
At the start: 18 parts, among them SW1 ChorusFilterPan, SW3 Chorus-FilterPan-B, SW5 ChorusFbInv, SW6 Chorus-Fb_Invert-B, U2 NJM4556

Commit message: assign footprints, start pcb
Other:
- note added: "- - -"
- note added: "- - - -"
- note added: "Aux2Fx\n SW"
- note added: "Chorus\nControl\n PCB"
- note added: "Chorus\nExtension\n PCB"
- note added: "Depth\n Pot"
- note added: "FbInv\n SW"
- note added: "Feedback\n Pot"
- note added: "FiltPan\n SW"
- note added: "KLM-598-3\n PCB"
- note added: "Keyboard Keys"
- note added: "LFOShape\n SW"
- note added: "Rate\n Pot"
- note added: "Stereo\n Pot"
- note added: "Synth2Fx\n SW"
- note added: "WetPass\n Pot"
- moved on the sheet: C11, C17, C20, C21, C48, C49, C51, C7, R12, R13, RV1, RV4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

Commit message: save-point before some experimental pcb markings
Parts:
- added JP31: Wet, symbol Jumper_Wire
- added JP32: Dry, symbol Jumper_Wire
- added JP33: FB, symbol Jumper_Wire
- added JP34: WetL, symbol Jumper_Wire
- added JP35: DryR, symbol Jumper_Wire
- added JP36: WetR, symbol Jumper_Wire
- added JP37: +A, symbol Jumper_Wire
- added JP38: GND, symbol Jumper_Wire
- added JP39: -A, symbol Jumper_Wire
- added JP41: SwR, symbol Jumper_Wire
- added JP42: SwL, symbol Jumper_Wire
- added JP43: WetLP, symbol Jumper_Wire
- added JP44: WetHP, symbol Jumper_Wire
- added JP45: WetNI, symbol Jumper_Wire
- added JP46: WetInv, symbol Jumper_Wire
- added JP47: ToHP, symbol Jumper_Wire
- added JP48: ToLP, symbol Jumper_Wire
- U2: symbol DualOpAmp -> Dual-Op-Amp
Connections:
- wire segments 89 -> 75
Other:
- note added: "Chorus-Ctrl PCB"
- note added: "Jumper wires JP31 - JP39\nconnect with pads P1 - P9\nrespectively on Chorus-Ext"
- note added: "Jumper wires JP41 - JP48\nconnect this Chorus-Ctrl\nboard to point to point wired\npanel controls"
- note removed: "Chorus-Control PCB"
- note removed: "Wet from \nremoved\nC20"
- moved on the sheet: C11, C17, C20, C21, C48, C49, C51, C7, R12, R13, RV1, RV4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

Commit message: routine  save-point
Parts:
- removed JP31: Wet, symbol Jumper_Wire
- removed JP32: Dry, symbol Jumper_Wire
- removed JP33: FB, symbol Jumper_Wire
- removed JP34: WetL, symbol Jumper_Wire
- removed JP35: DryR, symbol Jumper_Wire
- removed JP36: WetR, symbol Jumper_Wire
- removed JP37: +A, symbol Jumper_Wire
- removed JP38: GND, symbol Jumper_Wire
- removed JP39: -A, symbol Jumper_Wire
- removed JP41: SwR, symbol Jumper_Wire
- removed JP42: SwL, symbol Jumper_Wire
- removed JP43: WetLP, symbol Jumper_Wire
- removed JP44: WetHP, symbol Jumper_Wire
- removed JP45: WetNI, symbol Jumper_Wire
- removed JP46: WetInv, symbol Jumper_Wire
- removed JP47: ToHP, symbol Jumper_Wire
- removed JP48: ToLP, symbol Jumper_Wire
- removed SW1: ChorusFilterPan, symbol SW_DPDT_x2
- removed SW3: Chorus-FilterPan-B, symbol SW_DPDT_x2
- removed SW5: ChorusFbInv, symbol SW_DPDT_x2
- removed SW6: Chorus-Fb_Invert-B, symbol SW_DPDT_x2
- added P_+A_A6: red, MyKi_TH_Connectors:TH_Wire_Val, symbol F-M-Pins
- added P_-A_A8: brown, MyKi_TH_Connectors:TH_Wire_Val, symbol F-M-Pins
- added P_DryCP_A1, P_OnR_P3: orange, MyKi_TH_Connectors:TH_Wire_Val, symbol F-M-Pins
- added P_DryR_A3: orange+b, MyKi_TH_Connectors:TH_Wire_Val, symbol F-M-Pins
- added P_FB_A9: green, MyKi_TH_Connectors:TH_Wire_Val, symbol F-M-Pins
- added P_GND_A7: black, MyKi_TH_Connectors:TH_Wire_Val, symbol F-M-Pins
- added P_HP_P7: blue-b, MyKi_TH_Connectors:TH_Wire_Val, symbol F-M-Pins
- added P_LP_P8: purple-b, MyKi_TH_Connectors:TH_Wire_Val, symbol F-M-Pins
- added P_OnHP_P5, P_Wet_A5: blue, MyKi_TH_Connectors:TH_Wire_Val, symbol F-M-Pins
- added P_OnLP_P6, P_WetR_A4: purple, MyKi_TH_Connectors:TH_Wire_Val, symbol F-M-Pins
- added P_OnL_P4, P_WetL_A2: yellow, MyKi_TH_Connectors:TH_Wire_Val, symbol F-M-Pins
- added P_WetL_P2: yellow-b, MyKi_TH_Connectors:TH_Wire_Val, symbol F-M-Pins
- added P_WetR_P1: orange-b, MyKi_TH_Connectors:TH_Wire_Val, symbol F-M-Pins
- added SW1: ChoFilterPan, Buttons_Switches_THT:SW_CuK_JS202011AQN_DPDT_Angled, symbol DPDT
- added SW2: ChoFbInv, Buttons_Switches_THT:SW_CuK_JS202011AQN_DPDT_Angled, symbol DPDT
- C11, C17, C48, C49, C51: footprint (none) -> MyKi_TH_Capacitors:200Mil_TH_C
- C20: footprint (none) -> MyKi_TH_Capacitors:200Mil_TH_CP
- C21, C7: footprint (none) -> MyKi_TH_Capacitors:200Mil_TH_CP_no3D
- R12, R13: footprint (none) -> MyKi_TH_Resistors:400Mil_TH_Resistor
- RV1, RV4: footprint (none) -> MyKi_TH_Panel_Controls:400x200Mil_TH_Pot_Dual_FaceUp; symbol POT_Dual -> Dual_Pot
- RV6: footprint (none) -> MyKi_TH_Panel_Controls:400x500Mil_TH_Pot_reinfoced_FaceUp; symbol POT -> Pot
- U2: footprint MODULE -> MyKi_TH_IC:300Mil_DIP8
Connections:
- net at RV6.1 (G): no longer C51.1
- net at RV4.5 (W), RV6.2 (W): now also P_LP_P8.1 (B)
- net at RV6.3 (In): now also C51.1, P_FB_A9.1 (B)
- net at C48.1: now also P_HP_P7.1 (B)
- net at RV1.2 (W): now also P_WetL_A2.1 (B)
- net at RV1.3 (In): now also P_WetL_P2.1 (B)
- net at RV1.5 (W): now also P_DryR_A3.1 (B)
- net at RV1.6 (In): now also P_DryCP_A1.1 (B)
- net at C20.2: now also P_OnR_P3.1 (B)
- net at RV4.1 (G): now also P_OnL_P4.1 (B)
- net at C11.1, C7.1, U2.8 (V+): now also P_+A_A6.1 (B)
- net at C11.2, C17.2, C21.1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: now also P_GND_A7.1 (B)
- net at C17.1, C21.2, U2.4 (V-): now also P_-A_A8.1 (B)
- net at R13.1, U2.1 (←1), U2.2 (1-): now also P_OnHP_P5.1 (B)
- net at U2.3 (1+): now also P_Wet_A5.1 (B)
- net at R12.1, U2.7 (2→): now also P_OnLP_P6.1 (B)
- new net: P_WetR_A4.1 (B), P_WetR_P1.1 (B)
- new net: P_WetR_P1.2 (F), SW1.2 (C1)
- new net: P_WetL_P2.2 (F), SW1.5 (C2)
- new net: P_OnR_P3.2 (F), SW1.3 (on), SW1.4 (off)
- new net: P_OnL_P4.2 (F), SW1.1 (off), SW1.6 (on)
- new net: P_OnHP_P5.2 (F), SW2.3 (on), SW2.4 (off)
- new net: P_OnLP_P6.2 (F), SW2.1 (off), SW2.6 (on)
- new net: P_HP_P7.2 (F), SW2.2 (C1)
- new net: P_LP_P8.2 (F), SW2.5 (C2)
- new net +A_A6: P_+A_A6.2 (F)
- new net -A_A8: P_-A_A8.2 (F)
- new net DryCP_A1: P_DryCP_A1.2 (F)
- new net DryR_A3: P_DryR_A3.2 (F)
- new net FB_A9: P_FB_A9.2 (F)
- new net GND_A7: P_GND_A7.2 (F)
- new net WetL_A2: P_WetL_A2.2 (F)
- new net WetR_A4: P_WetR_A4.2 (F)
- new net Wet_A5: P_Wet_A5.2 (F)
Other:
- note added: "<- to LPF and \nFb (norm. Left)"
- note added: "Cho-Ctrl PCB"
- note added: "Header Pins P_*_P* connect directly\nbetween point to point wired panel \ncomponents arranged from the upper \nright corner of the synth downward."
- note added: "Pads P_*_A* run wires between this \nCho-Ctrl board and Cho-Ext."
- note removed: "- - -"
- note removed: "<- to LPF (norm.\nLeft) and Fb"
- note removed: "Chorus-Ctrl PCB"
- note removed: "Chorus\nExtension\n PCB"
- note removed: "Jumper wires JP31 - JP39\nconnect with pads P1 - P9\nrespectively on Chorus-Ext"
- note removed: "Jumper wires JP41 - JP48\nconnect this Chorus-Ctrl\nboard to point to point wired\npanel controls"
- note removed: "KLM-598-3\n PCB"
- note removed: "PCB mounted pots on\nChorus-Control PCB"
- moved on the sheet: C11, C17, C20, C21, C48, C49, C51, C7, R12, R13, U2
