File: old/Cho-Ctrl/Cho-Ctrl.kicad_pcb (KiCad board)
At the start: 2 copper layers, 34 parts, among them SW1 ChoFilterPan, SW2 ChoFbInv, U2 NJM4556

Commit message: Chorus mod effectively complete sans some clean up
Parts:
- removed PCB2: Cho-Ctrl, MyKi_TH_Board_Features:perfboard_single-sided_240x180Mil
- added REF**: Shunda 5CM*7CM (!), MyKi_TH_Board_Features:perfboard_24x18_Shunda_misprint, F.Cu at (240.3, 54.1)
- moved C11 56.1 mm to (227.6, 71.9)
- moved C17 56.1 mm to (222.5, 74.4)
- moved C20 56.1 mm to (245.4, 54.1)
- moved C21 56.1 mm to (225.0, 79.5)
- moved C48 56.1 mm to (240.3, 49.0)
- moved C49 56.1 mm to (245.4, 59.2)
- moved C51 56.1 mm to (245.4, 77.0)
- moved C7 56.1 mm to (225.0, 71.9)
- moved P_+A_A6 56.1 mm to (220.0, 71.9)
- moved P_-A_A8 56.1 mm to (217.4, 64.3)
- moved P_DryCP_A1 56.1 mm to (242.8, 33.8)
- moved P_DryR_A3 56.1 mm to (242.8, 28.7)
- moved P_FB_A9 56.1 mm to (245.4, 79.5)
- moved P_GND_A7 56.1 mm to (217.4, 79.5)
- moved P_HP_P7 56.1 mm to (240.3, 64.3)
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Routing:
- net /GND: track 161.5 -> 167.7 mm
Other:
- board text added: "blue"
- board text added: "blue-b"
- board text added: "orange"
- board text added: "orange-b"
- board text added: "purple"
- board text added: "purple-b"
- board text added: "yellow"
- board text added: "yellow-b"
