File: old/Cho-Ext/Cho-Ext.kicad_pcb (KiCad board)
At the start: 2 copper layers, 86 parts, among them J1 AuxAudioIn, SW3 AuxToChorus, SW4 KorgToChorus, SW5 LFO2 Sel, U1 TL084, X1 BackPlated_TH, X18 BackPlated_TH

Commit message: Chorus mod effectively complete sans some clean up
Parts:
- removed A1, A18, X1, X18: BackPlated_TH, MyKi_TH_Board_Features:BackPlated_TH
- removed Hole1, Hole2, Hole3, Hole4: 2mm_DrillHole, MyKi_TH_Board_Features:2mm_DrillHole
- added REF**: Shunda 5CM*7CM (!), MyKi_TH_Board_Features:perfboard_24x18_Shunda_misprint, F.Cu at (73.7, 66.0)
Other:
- board text removed: "1"
- board text removed: "10"
- board text removed: "11"
- board text removed: "12"
- board text removed: "13"
- board text removed: "14"
- board text removed: "15"
- board text removed: "16"
- board text removed: "17"
- board text removed: "18"
- board text removed: "2"
- board text removed: "3"
- board text removed: "4"
- board text removed: "5"
- board text removed: "6"
- board text removed: "7"
- board text removed: "8"
- board text removed: "9"
- board text removed: "A"
- board text removed: "B"
- board text removed: "C"
- board text removed: "Control-PCB"
- board text removed: "D"
- board text removed: "E"
- board text removed: "F"
- board text removed: "G"
- board text removed: "H"
- board text removed: "I"
- board text removed: "J"
- board text removed: "K"
- board text removed: "L"
- board text removed: "M"
- board text removed: "N"
- board text removed: "O"
- board text removed: "P"
- board text removed: "Q"
- board text removed: "R"
- board text removed: "S"
- board text removed: "T"
- board text removed: "U"
- board text removed: "V"
- board text removed: "W"
- board text removed: "X"
